Commit message: ik_mode updated

File: robots/olaf/olaf.urdf (robot description, URDF)
Before this commit: robot olaf, 16 links, 15 joints
Links:
- link left_foot_link: mass 0.5337193876053451 -> 0.24467; geometry collision mesh filename=meshes/left_foot.STL scale=0.001 0.001 0.001; visual mesh filename=meshes/left_foot.STL scale=0.001 0.001 0.001
- link left_foot_rotation: mass 0.6136768818052651 -> 0.80446; geometry collision mesh filename=meshes/left_foot_rotation.STL scale=0.001 0.001 0.001; visual mesh filename=meshes/left_foot_rotation.STL scale=0.001 0.001 0.001
- link left_hip: mass 0.5866748126521483 -> 0.5743; geometry collision mesh filename=meshes/left_hip.STL scale=0.001 0.001 0.001; visual mesh filename=meshes/left_hip.STL scale=0.001 0.001 0.001
- link left_hip_rotation: mass 0.5529873669984209 -> 0.72825; geometry collision mesh filename=meshes/left_hip_rotation.STL scale=0.001 0.001 0.001; visual mesh filename=meshes/left_hip_rotation.STL scale=0.001 0.001 0.001
- link left_shin: mass 0.5669545830968397 -> 0.5938; geometry collision mesh filename=meshes/left_shin.STL scale=0.001 0.001 0.001; visual mesh filename=meshes/left_shin.STL scale=0.001 0.001 0.001
- link left_thigh: mass 0.20336221361238202 -> 0.0617; geometry collision mesh filename=meshes/left_thigh.STL scale=0.001 0.001 0.001; visual mesh filename=meshes/left_thigh.STL scale=0.001 0.001 0.001
- link pelvis: mass 2.075931281689636 -> 6.42856; geometry collision mesh filename=meshes/pelvis.STL scale=0.001 0.001 0.001; visual mesh filename=meshes/pelvis.STL scale=0.001 0.001 0.001
- link right_foot_link: mass 0.5337193876053451 -> 0.24467; geometry collision mesh filename=meshes/right_foot.STL scale=0.001 0.001 0.001; visual mesh filename=meshes/right_foot.STL scale=0.001 0.001 0.001
- link right_foot_rotation: mass 0.6136768818052651 -> 0.80446; geometry collision mesh filename=meshes/right_foot_rotation.STL scale=0.001 0.001 0.001; visual mesh filename=meshes/right_foot_rotation.STL scale=0.001 0.001 0.001
- link right_hip: mass 0.5866748126521483 -> 0.5743; geometry collision mesh filename=meshes/right_hip.STL scale=0.001 0.001 0.001; visual mesh filename=meshes/right_hip.STL scale=0.001 0.001 0.001
- link right_hip_rotation: mass 0.5529873669984209 -> 0.72825; geometry collision mesh filename=meshes/right_hip_rotation.STL scale=0.001 0.001 0.001; visual mesh filename=meshes/right_hip_rotation.STL scale=0.001 0.001 0.001
- link right_shin: mass 0.5669545830968397 -> 0.5938; geometry collision mesh filename=meshes/right_shin.STL scale=0.001 0.001 0.001; visual mesh filename=meshes/right_shin.STL scale=0.001 0.001 0.001
- link right_thigh: mass 0.20336221361238202 -> 0.0617; geometry collision mesh filename=meshes/right_thigh.STL scale=0.001 0.001 0.001; visual mesh filename=meshes/right_thigh.STL scale=0.001 0.001 0.001
Joints:
- joint left_ankle_pitch: axis -0.0 1.0 0.0 -> 0 -1 0; limit lower=-1.57 upper=1.57 effort=23.7 velocity=30 -> lower=-0.7853982 upper=1.5707963 effort=24.0 velocity=5; origin xyz=4.3e-05 0.004601 -0.08575 rpy=0 0 0 -> xyz=0 -0.0024 -0.09 rpy=0 0 0
- joint left_ankle_roll: axis 1.0 0.0 0.0 -> 1 0 0; limit lower=-3.14 upper=3.14 effort=23.7 velocity=30 -> lower=-0.7853982 upper=0.7853982 effort=24.0 velocity=5; origin xyz=-0.015764 -0.012761 -0.044999 rpy=0 0 0 -> xyz=0.0265 -0.0077 -0.0655 rpy=0 0 0
- joint left_foot_frame: origin xyz=0.0 0.0 0.0 rpy=0 0 0 -> xyz=-0.0265 0.0 -0.052 rpy=0 0 0
- joint left_hip_pitch: axis 0.0 -1.0 0.0 -> 0 1 0; limit lower=-1.57 upper=1.57 effort=23.7 velocity=30 -> lower=-1.3089969 upper=0.2617994 effort=23.7 velocity=30; origin xyz=0.05675 0.01945 -0.011502 rpy=0 0 0 -> xyz=0.0537 0.0051 0.0 rpy=0 0 0
- joint left_hip_roll: axis 1.0 -0.0 0.0 -> 1 0 0; limit lower=-1.57 upper=0.7853982 effort=23.7 velocity=30 -> lower=-0.7853982 upper=0.7853982 effort=23.7 velocity=30; origin xyz=-0.0564 1e-06 -0.05575 rpy=0 0 0 -> xyz=-0.0537 0.0 -0.072 rpy=0 0 0
- joint left_hip_yaw: axis 0.0 0.0 1.0 -> 0 0 -1; origin xyz=-0.000138 0.055638 0.3 rpy=0 0 0 -> xyz=0 0.07 0.3439 rpy=0 0 0
- joint left_knee: axis 0.0 -1.0 0.0 -> 0 1 0; limit lower=-1.57 upper=1.57 effort=23.7 velocity=30 -> lower=0.0 upper=2.1816624 effort=23.7 velocity=30; origin xyz=-3e-06 0.005001 -0.07 rpy=0 0 0 -> xyz=0 0.005 -0.0644 rpy=0 0 0
- joint right_ankle_pitch: axis 0.0 -1.0 0.0 -> 0 -1 0; limit lower=-1.57 upper=1.57 effort=23.7 velocity=30 -> lower=-0.7853982 upper=1.5707963 effort=24.0 velocity=5; origin xyz=-4.3e-05 -0.004601 -0.08575 rpy=0 0 0 -> xyz=0 -0.0024 -0.09 rpy=0 0 0
- joint right_ankle_roll: axis -1.0 0.0 0.0 -> 1 0 0; limit lower=-3.14 upper=3.14 effort=23.7 velocity=30 -> lower=-0.7853982 upper=0.7853982 effort=24.0 velocity=5; origin xyz=0.015764 0.012761 -0.044999 rpy=0 0 0 -> xyz=0.0265 -0.0077 -0.0655 rpy=0 0 0
- joint right_foot_frame: origin xyz=0.0 0.0 0.0 rpy=0 0 0 -> xyz=-0.0265 0.0 -0.052 rpy=0 0 0
- joint right_hip_pitch: axis -0.0 -1.0 1.3e-05 -> 0 1 0; limit lower=-1.57 upper=1.57 effort=23.7 velocity=30 -> lower=-1.3089969 upper=0.2617994 effort=23.7 velocity=30; origin xyz=-0.056751 -0.01945 -0.011502 rpy=0 0 0 -> xyz=0.0537 0.0051 0.0 rpy=0 0 0
- joint right_hip_roll: axis -1.0 0.0 -0.0 -> 1 0 0; limit lower=-1.57 upper=0.7853982 effort=23.7 velocity=30 -> lower=-0.7853982 upper=0.7853982 effort=23.7 velocity=30; origin xyz=0.0564 0.0 -0.05575 rpy=0 0 0 -> xyz=-0.0537 0.0 -0.072 rpy=0 0 0
- joint right_hip_yaw: axis -0.0 0.0 1.0 -> 0 0 -1; origin xyz=-0.001138 -0.054362 0.3 rpy=0 0 0 -> xyz=0 -0.07 0.3439 rpy=0 0 3.14159265359
- joint right_knee: axis 0.0 -1.0 0.0 -> 0 1 0; limit lower=-1.57 upper=1.57 effort=23.7 velocity=30 -> lower=0.0 upper=2.1816624 effort=23.7 velocity=30; origin xyz=3e-06 -0.005001 -0.07 rpy=0 0 0 -> xyz=0 0.005 -0.0644 rpy=0 0 0
- joint trunk_frame: origin xyz=0.0 0.0 0.3 rpy=0 0 0 -> xyz=0 0 0.3505 rpy=0 0 0
